Commit message: 完成具身任务闭环

File: src/x_bot/urdf/gz.xacro (robot description, xacro)
@@ -1,4 +1,7 @@
 <?xml version="1.0"?>
 <robot xmlns:xacro="http://www.ros.org/wiki/xacro" name="x_bot">
+    <!-- 探索+Cartographer 时必须为 false，否则会与 Cartographer 争抢 odom→base_footprint TF -->
+    <xacro:arg name="publish_odom_tf" default="false"/>
+    <xacro:property name="publish_odom_tf" value="$(arg publish_odom_tf)"/>
     <!-- ........................... SENSOR PLUGIN ................................... -->
     <gazebo>
@@ -41,6 +44,8 @@
             <robot_base_frame>base_footprint</robot_base_frame>
             <odom_topic>x_bot/odom</odom_topic>
-            <!-- 禁用 TF 发布，由 Cartographer 或其他 SLAM 系统提供 -->
-            <!-- <tf_topic>/tf</tf_topic> -->
+            <!-- 仅导航(AMCL)模式开启；Cartographer 模式由 SLAM 发布 odom→base -->
+            <xacro:if value="${publish_odom_tf}">
+            <tf_topic>/tf</tf_topic>
+            </xacro:if>
             <dimensions>2</dimensions>
             <odom_publish_frequency>50</odom_publish_frequency>
