Commit message: 修复地盘运动问题

File: src/x_bot/urdf/x_bot.xacro (robot description, xacro)
@@ -39,4 +39,6 @@
     <xacro:arg name="sim_gz" default="false" />
     <xacro:arg name="sim_isaac" default="false" />
+    <xacro:arg name="mid360_xyz" default="0.25 0 0.0875" />
+    <xacro:arg name="mid360_rpy" default="0 0 0" />
     <xacro:arg name="odometry_source" default="world" />
     <xacro:property name="odometry_source" value="$(arg odometry_source)"/>
@@ -92,4 +94,5 @@
     <xacro:traction_wheel cardinality="back" dexterity="right" origin_x="-${traction_wheel_base/2}" origin_y="-${traction_track_width/2}" origin_z="-${chassis_height/2+traction_wheel_radius*0.5}"/>
     <!-- ............................. 2D LIDAR ........................................ -->
+    <xacro:unless value="$(arg sim_isaac)">
     <xacro:if value="$(arg two_d_lidar_enabled)">
         <link name="two_d_lidar">
@@ -122,5 +125,29 @@
         </gazebo>
     </xacro:if>
-    <!-- ............................. IMU ........................................ -->
+    </xacro:unless>
+    <!-- Isaac-only roof sensor. IMU and optical origin are colocated in simulation. -->
+    <xacro:if value="$(arg sim_isaac)">
+        <link name="mid360_link">
+            <visual><geometry><box size="0.065 0.065 0.060"/></geometry><material name="black"/></visual>
+            <collision><geometry><box size="0.065 0.065 0.060"/></geometry></collision>
+            <!-- 50 mm standoff below the sensor housing. -->
+            <visual><origin xyz="0 0 -0.055"/><geometry><box size="0.020 0.020 0.050"/></geometry><material name="black"/></visual>
+            <collision><origin xyz="0 0 -0.055"/><geometry><box size="0.020 0.020 0.050"/></geometry></collision>
+            <inertial>
+                <mass value="0.265"/>
+                <inertia ixx="0.00017280" ixy="0" ixz="0" iyy="0.00017280" iyz="0" izz="0.00018660"/>
+            </inertial>
+        </link>
+        <joint name="mid360_joint" type="fixed">
+            <parent link="roof_link"/><child link="mid360_link"/>
+            <origin xyz="$(arg mid360_xyz)" rpy="$(arg mid360_rpy)"/>
+        </joint>
+        <link name="mid360_imu_link"/>
+        <joint name="mid360_imu_joint" type="fixed">
+            <parent link="mid360_link"/><child link="mid360_imu_link"/>
+            <origin xyz="0 0 0" rpy="0 0 0"/>
+        </joint>
+    </xacro:if>
+    <!-- Legacy Gazebo IMU frame is retained for backend compatibility. -->
     <link name="imu_frame"/>
     <joint name="imu_joint" type="fixed">

Commit message: fix: stabilize Isaac base and enable default auto exploration

File: src/x_bot/urdf/x_bot.xacro (robot description, xacro)
@@ -57,9 +57,26 @@
     <!-- ................................ BASE LINK .................................. -->
     <link name="base_footprint"/>
-    <link name="base_link"/>
+    <link name="base_link">
+        <!-- Give Isaac a physical root above both chassis and wheel branches. -->
+        <xacro:if value="$(arg sim_isaac)">
+            <inertial>
+                <!-- A tiny root body is ill-conditioned against the 70 kg
+                     chassis. Allocate 1 kg of chassis mass to the root. -->
+                <mass value="1"/>
+                <xacro:cylinder_inertia m="1" r="${chassis_radius}" h="${chassis_height}"/>
+            </inertial>
+        </xacro:if>
+    </link>
     <joint name="base_joint" type="fixed">
         <parent link="base_footprint"/>
         <child link="base_link"/>
-        <origin xyz="0.0 0 ${chassis_height/2 + traction_wheel_radius}" rpy="0 0 0.0" />
+        <!-- Isaac spawns base_footprint on z=0: wheel centres must be one
+             radius above that plane (wheel joints are 0.09 m below base_link). -->
+        <xacro:if value="$(arg sim_isaac)">
+            <origin xyz="0 0 ${chassis_height/2 + 1.5*traction_wheel_radius}" rpy="0 0 0"/>
+        </xacro:if>
+        <xacro:unless value="$(arg sim_isaac)">
+            <origin xyz="0.0 0 ${chassis_height/2 + traction_wheel_radius}" rpy="0 0 0.0" />
+        </xacro:unless>
     </joint>
     <link name="chassis_link">
@@ -78,6 +95,12 @@
         </visual>
         <inertial>
-            <mass value="${chassis_mass}" />
-            <xacro:cylinder_inertia m="${chassis_mass}" r="${chassis_radius}" h="${chassis_height}"/>
+            <xacro:if value="$(arg sim_isaac)">
+                <mass value="${chassis_mass-1}"/>
+                <xacro:cylinder_inertia m="${chassis_mass-1}" r="${chassis_radius}" h="${chassis_height}"/>
+            </xacro:if>
+            <xacro:unless value="$(arg sim_isaac)">
+                <mass value="${chassis_mass}" />
+                <xacro:cylinder_inertia m="${chassis_mass}" r="${chassis_radius}" h="${chassis_height}"/>
+            </xacro:unless>
         </inertial>
     </link>
@@ -193,4 +216,11 @@
             <material name="grey"/>
         </visual>
+        <xacro:if value="$(arg sim_isaac)">
+            <collision>
+                <geometry>
+                    <cylinder radius="0.02" length="0.08"/>
+                </geometry>
+            </collision>
+        </xacro:if>
     </link>
     <joint name="pillar_fl_joint" type="fixed">
@@ -208,4 +238,11 @@
             <material name="grey"/>
         </visual>
+        <xacro:if value="$(arg sim_isaac)">
+            <collision>
+                <geometry>
+                    <cylinder radius="0.02" length="0.08"/>
+                </geometry>
+            </collision>
+        </xacro:if>
     </link>
     <joint name="pillar_fr_joint" type="fixed">
@@ -223,4 +260,11 @@
             <material name="grey"/>
         </visual>
+        <xacro:if value="$(arg sim_isaac)">
+            <collision>
+                <geometry>
+                    <cylinder radius="0.02" length="0.08"/>
+                </geometry>
+            </collision>
+        </xacro:if>
     </link>
     <joint name="pillar_bl_joint" type="fixed">
@@ -238,4 +282,11 @@
             <material name="grey"/>
         </visual>
+        <xacro:if value="$(arg sim_isaac)">
+            <collision>
+                <geometry>
+                    <cylinder radius="0.02" length="0.08"/>
+                </geometry>
+            </collision>
+        </xacro:if>
     </link>
     <joint name="pillar_br_joint" type="fixed">
@@ -293,4 +344,5 @@
             robot_type="fr3"
             parent="fr3_mount_link"
+            connected_to=""
             xyz="0 0 0"
             rpy="0 0 0"
@@ -306,4 +358,11 @@
             dynamics="${xacro.load_yaml('$(find franka_description)/robots/fr3/dynamics.yaml')}"
         />
+        <!-- With gazebo=false, the Franka macro does not use parent and would
+             otherwise create a disconnected default base link. -->
+        <joint name="fr3_base_joint" type="fixed">
+            <parent link="fr3_mount_link"/>
+            <child link="fr3_link0"/>
+            <origin xyz="0 0 0" rpy="0 0 0"/>
+        </joint>
     </xacro:if>
     <xacro:unless value="$(arg sim_isaac)">
