Commit message: Simplify workspace layout and launchers, streamline manipulation and improve turning

File: src/robot/x_bot/urdf/materials.xacro (robot description, xacro)
@@ -3,4 +3,7 @@
     <material name="black">
         <color rgba="0.0 0.0 0.0 1.0"/>
+    </material>
+    <material name="lidar_silver">
+        <color rgba="0.82 0.84 0.87 1.0"/>
     </material>
     <material name="blue">

File: src/robot/x_bot/urdf/x_bot.xacro (robot description, xacro)
@@ -153,8 +153,8 @@
     <xacro:if value="${'$(arg sim_isaac)' == 'true' or '$(arg mid360_enabled)' == 'true'}">
         <link name="mid360_link">
-            <visual><geometry><box size="0.065 0.065 0.060"/></geometry><material name="black"/></visual>
+            <visual><geometry><box size="0.065 0.065 0.060"/></geometry><material name="lidar_silver"/></visual>
             <collision><geometry><box size="0.065 0.065 0.060"/></geometry></collision>
             <!-- 50 mm standoff below the sensor housing. -->
-            <visual><origin xyz="0 0 -0.055"/><geometry><box size="0.020 0.020 0.050"/></geometry><material name="black"/></visual>
+            <visual><origin xyz="0 0 -0.055"/><geometry><box size="0.020 0.020 0.050"/></geometry><material name="lidar_silver"/></visual>
             <collision><origin xyz="0 0 -0.055"/><geometry><box size="0.020 0.020 0.050"/></geometry></collision>
             <inertial>
